File: neuromorphic-ir-event-sensor.kicad_pcb (KiCad board)
At the start: 2 copper layers, 50 x 70 mm, 92 parts, among them Q1 AO3400A

Commit message: fix(pcb): correct LED1 pinout, complete routing, and regenerate manufacturing package
- Correct TSAL6200 IR LED pinout (Pad 1 Cathode -> LED_K, Pad 2 Anode -> 3V3) in schematic and PCB layout
- Complete copper routing with 0 DRC violations and 0 unconnected nets
- Re-export all production Gerbers, Excellon drill files, and revA ZIP archive
- Regenerate 3D CAD STEP model and documentation vector SVGs (PCB 2D & schematic)
Connections:
- LED1 pad 1: (no net) -> LED_K
- LED1 pad 2: LED_K -> 3V3
Routing:
- net LED_K: track 9.65 -> 5.77 mm
