File: neuromorphic-ir-event-sensor.kicad_pcb (KiCad board)
At the start: 2 copper layers, 50 x 70 mm, 92 parts, among them Q1 AO3400A

Commit message: Promote verified Rev A candidate to main KiCad project
Parts:
- removed CA1, CA2, CA3, CA4, CREF2, C_DEC_CMP1, C_DEC_CMP2, C_DEC_CMP3, C_DEC_CMP4, C_DEC_TIA1, C_DEC_TIA2, C_DEC_TIA3, C_DEC_TIA4: 100nF, Capacitor_SMD:C_0603_1608Metric
- removed CF1, CF2, CF3, CF4: 47pF, Capacitor_SMD:C_0603_1608Metric
- removed COS_OFF_BL, COS_OFF_BR, COS_OFF_TL, COS_OFF_TR, COS_ON_BL, COS_ON_BR, COS_ON_TL, COS_ON_TR: 12nF, Capacitor_SMD:C_0603_1608Metric
- removed CREF1: 1uF, Capacitor_SMD:C_0603_1608Metric
- removed C_BULK_A, C_BULK_D, C_LED: 10uF, Capacitor_SMD:C_0805_2012Metric
- removed DPD1, DPD2, DPD3, DPD4: VBPW34FASR, OptoDevice:Osram_BPW34S-SMD
- removed H (x4): M3, MountingHole:MountingHole_3.2mm_M3
- removed H (x2): M2, MountingHole:MountingHole_2.2mm_M2
- removed J_DEBUG: Analog_Debug, Connector_PinHeader_2.54mm:PinHeader_1x06_P2.54mm_Vertical
- removed J_FPGA: Tang_Nano_Event_Out, Connector_PinHeader_2.54mm:PinHeader_2x05_P2.54mm_Vertical
- removed LED1: TSAL6200, LED_THT:LED_D5.0mm
- removed RA1, RA2, RA3, RA4: 22k, Resistor_SMD:R_0603_1608Metric
- removed RF1, RF2, RF3, RF4: 18.0k, Resistor_SMD:R_0603_1608Metric
- removed RG: 100R, Resistor_SMD:R_0603_1608Metric
- removed RLED: 82R, Resistor_SMD:R_1206_3216Metric
- removed ROS_OFF_BL, ROS_OFF_BR, ROS_OFF_TL, ROS_OFF_TR, ROS_ON_BL, ROS_ON_BR, ROS_ON_TL, ROS_ON_TR: 8.2k, Resistor_SMD:R_0603_1608Metric
- removed ROUT_OFF_BL, ROUT_OFF_BR, ROUT_OFF_TL, ROUT_OFF_TR, ROUT_ON_BL, ROUT_ON_BR, ROUT_ON_TL, ROUT_ON_TR: 150R, Resistor_SMD:R_0603_1608Metric
- removed RPD: 100k, Resistor_SMD:R_0603_1608Metric
- removed RTHN_A: 301k, Resistor_SMD:R_0603_1608Metric
- removed RTHN_B, RTHP_B: 10.0k, Resistor_SMD:R_0603_1608Metric
- removed RTHP_A: 499k, Resistor_SMD:R_0603_1608Metric
- removed U_CMP1, U_CMP2, U_CMP3, U_CMP4: TLV3202, Package_SO:SOIC-8_3.9x4.9mm_P1.27mm
- removed U_OS_OFF_BL, U_OS_OFF_BR, U_OS_OFF_TL, U_OS_OFF_TR, U_OS_ON_BL, U_OS_ON_BR, U_OS_ON_TL, U_OS_ON_TR: 74LVC1G123, Package_SO:VSSOP-8_2.3x2mm_P0.5mm
- removed U_REF: REF3312, Package_TO_SOT_SMD:SOT-23-3
- removed U_TIA1, U_TIA2, U_TIA3, U_TIA4: OPA381, Package_SO:MSOP-8_3x3mm_P0.65mm
- added C1: 47pF, Capacitor_SMD:C_0603_1608Metric, F.Cu at (116.5, 105.0)
- added C10: 100nF, Capacitor_SMD:C_0603_1608Metric, F.Cu at (137.9, 107.0)
- added C11: 100nF, Capacitor_SMD:C_0603_1608Metric, F.Cu at (110.5, 127.5)
- added C12: 100nF, Capacitor_SMD:C_0603_1608Metric, F.Cu at (135.4, 123.0)
- added C13: 100nF, Capacitor_SMD:C_0603_1608Metric, F.Cu at (104.5, 123.0)
- added C14: 100nF, Capacitor_SMD:C_0603_1608Metric, F.Cu at (144.4, 113.5)
- added C15: 100nF, Capacitor_SMD:C_0603_1608Metric, F.Cu at (102.0, 133.9)
- added C16: 100nF, Capacitor_SMD:C_0603_1608Metric, F.Cu at (144.4, 128.0)
- added C17: 12nF, Capacitor_SMD:C_0603_1608Metric, F.Cu at (111.0, 152.4)
- added C18: 12nF, Capacitor_SMD:C_0603_1608Metric, F.Cu at (108.0, 160.4)
- added C19: 12nF, Capacitor_SMD:C_0603_1608Metric, F.Cu at (122.5, 152.4)
- added C2: 47pF, Capacitor_SMD:C_0603_1608Metric, F.Cu at (133.9, 105.0)
- added C20: 12nF, Capacitor_SMD:C_0603_1608Metric, F.Cu at (123.0, 158.9)
- added C21: 12nF, Capacitor_SMD:C_0603_1608Metric, F.Cu at (134.4, 152.4)
- added C22: 12nF, Capacitor_SMD:C_0603_1608Metric, F.Cu at (131.9, 160.4)
- added C23: 12nF, Capacitor_SMD:C_0603_1608Metric, F.Cu at (145.9, 152.4)
- added C24: 12nF, Capacitor_SMD:C_0603_1608Metric, F.Cu at (143.4, 160.4)
- added C25: 1uF, Capacitor_SMD:C_0603_1608Metric, F.Cu at (121.0, 104.5)
- added C26: 100nF, Capacitor_SMD:C_0603_1608Metric, F.Cu at (121.0, 102.5)
- added C27: 10uF, Capacitor_SMD:C_0805_2012Metric, F.Cu at (116.5, 102.0)
- added C28: 10uF, Capacitor_SMD:C_0805_2012Metric, F.Cu at (128.9, 103.0)
- added C29: 10uF, Capacitor_SMD:C_0805_2012Metric, F.Cu at (132.9, 102.5)
- added C3: 47pF, Capacitor_SMD:C_0603_1608Metric, F.Cu at (116.5, 123.5)
- added C30: 100nF, Capacitor_SMD:C_0603_1608Metric, F.Cu at (108.5, 149.4)
- added C31: 100nF, Capacitor_SMD:C_0603_1608Metric, F.Cu at (111.5, 156.9)
- added C32: 100nF, Capacitor_SMD:C_0603_1608Metric, F.Cu at (120.0, 149.4)
- added C33: 100nF, Capacitor_SMD:C_0603_1608Metric, F.Cu at (123.0, 156.9)
- added C34: 100nF, Capacitor_SMD:C_0603_1608Metric, F.Cu at (131.9, 149.4)
- added C35: 100nF, Capacitor_SMD:C_0603_1608Metric, F.Cu at (134.9, 156.9)
- added C36: 100nF, Capacitor_SMD:C_0603_1608Metric, F.Cu at (143.4, 149.4)
- added C37: 100nF, Capacitor_SMD:C_0603_1608Metric, F.Cu at (146.4, 156.9)
- added C4: 47pF, Capacitor_SMD:C_0603_1608Metric, F.Cu at (132.9, 129.9)
- added C5: 100nF, Capacitor_SMD:C_0603_1608Metric, F.Cu at (110.5, 111.0)
- added C6: 100nF, Capacitor_SMD:C_0603_1608Metric, F.Cu at (139.4, 111.0)
- added C7: 100nF, Capacitor_SMD:C_0603_1608Metric, F.Cu at (110.5, 123.5)
- added C8: 100nF, Capacitor_SMD:C_0603_1608Metric, F.Cu at (139.4, 123.5)
- added C9: 100nF, Capacitor_SMD:C_0603_1608Metric, F.Cu at (111.5, 108.0)
- added D1: VBPW34S, VBPW34S:XDCR_VBPW34S, F.Cu at (121.9, 111.9)
- added D2: VBPW34S, VBPW34S:XDCR_VBPW34S, F.Cu at (127.4, 111.9)
- added D3: VBPW34S, VBPW34S:XDCR_VBPW34S, F.Cu at (121.9, 122.8)
- added D4: VBPW34S, VBPW34S:XDCR_VBPW34S, F.Cu at (127.4, 122.8)
- added D5: TSAL6200, LED_THT:LED_D5.0mm, F.Cu at (124.7, 135.1)
- added H1: MountingHole, MountingHole:MountingHole_3.2mm_M3, F.Cu at (103.6, 103.7)
- added H2: MountingHole, MountingHole:MountingHole_3.2mm_M3, F.Cu at (145.6, 103.7)
- added H3: MountingHole, MountingHole:MountingHole_3.2mm_M3, F.Cu at (103.6, 165.7)
- added H4: MountingHole, MountingHole:MountingHole_3.2mm_M3, F.Cu at (145.6, 165.7)
- added H5: MountingHole, MountingHole:MountingHole_2.2mm_M2, F.Cu at (114.7, 117.7)
- added H6: MountingHole, MountingHole:MountingHole_2.2mm_M2, F.Cu at (134.7, 117.7)
- added J1: FPGA_Events_2x5, Connector_PinHeader_2.54mm:PinHeader_2x05_P2.54mm_Vertical, F.Cu at (111.8, 165.9)
- added J2: Analog_Debug, Connector_PinHeader_2.54mm:PinHeader_1x06_P2.54mm_Vertical, F.Cu at (126.3, 164.7)
- added J3: LED_Enable_Input, Connector_PinHeader_2.54mm:PinHeader_1x02_P2.54mm_Vertical, F.Cu at (143.7, 138.4)
- added R1: 18.0k, Resistor_SMD:R_0603_1608Metric, F.Cu at (115.5, 111.5)
- added R10: 8.2k, Resistor_SMD:R_0603_1608Metric, F.Cu at (111.5, 158.9)
- added R11: 8.2k, Resistor_SMD:R_0603_1608Metric, F.Cu at (118.0, 149.4)
- added R12: 8.2k, Resistor_SMD:R_0603_1608Metric, F.Cu at (115.0, 156.4)
- added R13: 8.2k, Resistor_SMD:R_0603_1608Metric, F.Cu at (129.9, 149.4)
- added R14: 8.2k, Resistor_SMD:R_0603_1608Metric, F.Cu at (135.4, 158.9)
- added R15: 8.2k, Resistor_SMD:R_0603_1608Metric, F.Cu at (141.4, 149.4)
- added R16: 8.2k, Resistor_SMD:R_0603_1608Metric, F.Cu at (146.9, 158.9)
- added R17: 150R, Resistor_SMD:R_0603_1608Metric, F.Cu at (110.5, 148.9)
- added R18: 150R, Resistor_SMD:R_0603_1608Metric, F.Cu at (104.5, 160.4)
- added R19: 150R, Resistor_SMD:R_0603_1608Metric, F.Cu at (122.0, 148.9)
- added R2: 18.0k, Resistor_SMD:R_0603_1608Metric, F.Cu at (132.9, 111.5)
- added R20: 150R, Resistor_SMD:R_0603_1608Metric, F.Cu at (126.5, 158.4)
- added R21: 150R, Resistor_SMD:R_0603_1608Metric, F.Cu at (133.9, 148.9)
- added R22: 150R, Resistor_SMD:R_0603_1608Metric, F.Cu at (128.4, 160.4)
- added R23: 150R, Resistor_SMD:R_0603_1608Metric, F.Cu at (145.4, 148.9)
- added R24: 150R, Resistor_SMD:R_0603_1608Metric, F.Cu at (139.9, 160.4)
- added R25: 82R, Resistor_SMD:R_1206_3216Metric, F.Cu at (118.5, 132.4)
- added R26: 100R, Resistor_SMD:R_0603_1608Metric, F.Cu at (101.5, 137.4)
- added R27: 100k, Resistor_SMD:R_0603_1608Metric, F.Cu at (103.5, 141.4)
- added R28: 499k, Resistor_SMD:R_0603_1608Metric, F.Cu at (136.9, 102.5)
- added R29: 10.0k, Resistor_SMD:R_0603_1608Metric, F.Cu at (140.4, 102.5)
- added R3: 18.0k, Resistor_SMD:R_0603_1608Metric, F.Cu at (115.5, 129.9)
- added R30: 10.0k, Resistor_SMD:R_0603_1608Metric, F.Cu at (109.5, 104.5)
- added R31: 301k, Resistor_SMD:R_0603_1608Metric, F.Cu at (113.0, 104.5)
- added R32: 2.0M, Resistor_SMD:R_0603_1608Metric, F.Cu at (113.0, 121.5)
- added R33: 2.0M, Resistor_SMD:R_0603_1608Metric, F.Cu at (102.0, 118.0)
- added R34: 2.0M, Resistor_SMD:R_0603_1608Metric, F.Cu at (142.4, 113.5)
- added R35: 2.0M, Resistor_SMD:R_0603_1608Metric, F.Cu at (147.4, 118.5)
- added R36: 2.0M, Resistor_SMD:R_0603_1608Metric, F.Cu at (109.5, 137.4)
- added R37: 2.0M, Resistor_SMD:R_0603_1608Metric, F.Cu at (102.0, 130.4)
- added R38: 2.0M, Resistor_SMD:R_0603_1608Metric, F.Cu at (140.4, 128.4)
- added R39: 2.0M, Resistor_SMD:R_0603_1608Metric, F.Cu at (147.4, 130.9)
- added R4: 18.0k, Resistor_SMD:R_0603_1608Metric, F.Cu at (132.4, 123.5)
- added R40: 10.0k, Resistor_SMD:R_0603_1608Metric, F.Cu at (104.5, 113.5)
- added R41: 10.0k, Resistor_SMD:R_0603_1608Metric, F.Cu at (144.4, 123.0)
- added R42: 10.0k, Resistor_SMD:R_0603_1608Metric, F.Cu at (104.5, 128.0)
- added R43: 10.0k, Resistor_SMD:R_0603_1608Metric, F.Cu at (147.4, 135.4)
- added R5: 22k, Resistor_SMD:R_0603_1608Metric, F.Cu at (110.5, 113.0)
- added R6: 22k, Resistor_SMD:R_0603_1608Metric, F.Cu at (139.4, 113.0)
- added R7: 22k, Resistor_SMD:R_0603_1608Metric, F.Cu at (110.5, 125.5)
- added R8: 22k, Resistor_SMD:R_0603_1608Metric, F.Cu at (139.4, 125.5)
- added R9: 8.2k, Resistor_SMD:R_0603_1608Metric, F.Cu at (106.5, 149.4)
- added TP1: VTH_ON, TestPoint:TestPoint_Pad_D1.0mm, F.Cu at (113.0, 102.0)
- added TP10: RAW_OFF_BR, TestPoint:TestPoint_Pad_D1.0mm, F.Cu at (140.5, 105.5)
- added TP2: VTH_OFF, TestPoint:TestPoint_Pad_D1.0mm, F.Cu at (140.4, 108.0)
- added TP3: RAW_ON_TL, TestPoint:TestPoint_Pad_D1.0mm, F.Cu at (107.5, 122.5)
- added TP4: RAW_OFF_TL, TestPoint:TestPoint_Pad_D1.0mm, F.Cu at (143.0, 109.0)
- added TP5: RAW_ON_TR, TestPoint:TestPoint_Pad_D1.0mm, F.Cu at (109.0, 107.0)
- added TP6: RAW_OFF_TR, TestPoint:TestPoint_Pad_D1.0mm, F.Cu at (136.0, 113.5)
- added TP7: RAW_ON_BL, TestPoint:TestPoint_Pad_D1.0mm, F.Cu at (102.0, 109.0)
- added TP8: RAW_OFF_BL, TestPoint:TestPoint_Pad_D1.0mm, F.Cu at (104.5, 109.0)
- added TP9: RAW_ON_BR, TestPoint:TestPoint_Pad_D1.0mm, F.Cu at (107.0, 109.5)
- added U1: OPA381AIDGKR, Package_SO:MSOP-8_3x3mm_P0.65mm, F.Cu at (115.9, 108.2)
- added U10: SN74LVC1G123DCU, Package_SO:VSSOP-8_2.3x2mm_P0.5mm, F.Cu at (107.2, 157.7)
- added U11: SN74LVC1G123DCU, Package_SO:VSSOP-8_2.3x2mm_P0.5mm, F.Cu at (118.7, 152.7)
- added U12: SN74LVC1G123DCU, Package_SO:VSSOP-8_2.3x2mm_P0.5mm, F.Cu at (118.7, 157.7)
- added U13: SN74LVC1G123DCU, Package_SO:VSSOP-8_2.3x2mm_P0.5mm, F.Cu at (130.7, 152.7)
- added U14: SN74LVC1G123DCU, Package_SO:VSSOP-8_2.3x2mm_P0.5mm, F.Cu at (130.7, 157.7)
- added U15: SN74LVC1G123DCU, Package_SO:VSSOP-8_2.3x2mm_P0.5mm, F.Cu at (142.2, 152.7)
- added U16: SN74LVC1G123DCU, Package_SO:VSSOP-8_2.3x2mm_P0.5mm, F.Cu at (142.2, 157.7)
- added U17: REF3312AIDBZR, Package_TO_SOT_SMD:SOT-23-3, F.Cu at (125.0, 103.5)
- added U2: OPA381AIDGKR, Package_SO:MSOP-8_3x3mm_P0.65mm, F.Cu at (133.4, 108.2)
- added U3: OPA381AIDGKR, Package_SO:MSOP-8_3x3mm_P0.65mm, F.Cu at (115.9, 126.7)
- added U4: OPA381AIDGKR, Package_SO:MSOP-8_3x3mm_P0.65mm, F.Cu at (133.4, 126.7)
- added U5: TLV3202AIDR, Package_SO:SOIC-8_3.9x4.9mm_P1.27mm, F.Cu at (107.2, 118.2)
- added U6: TLV3202AIDR, Package_SO:SOIC-8_3.9x4.9mm_P1.27mm, F.Cu at (142.2, 118.2)
- added U7: TLV3202AIDR, Package_SO:SOIC-8_3.9x4.9mm_P1.27mm, F.Cu at (107.2, 132.7)
- added U8: TLV3202AIDR, Package_SO:SOIC-8_3.9x4.9mm_P1.27mm, F.Cu at (142.2, 132.7)
- added U9: SN74LVC1G123DCU, Package_SO:VSSOP-8_2.3x2mm_P0.5mm, F.Cu at (107.2, 152.7)
- moved FB1 137.1 mm to (109.5, 102.5)
- moved Q1 128.5 mm to (104.6, 137.6)
Connections:
- FB1 pad 1: 3V3 -> /3V3
- FB1 pad 2: 3V3_ANALOG -> /3V3_ANALOG
- Q1 pad 1: LED_GATE -> /LED_GATE
- Q1 pad 2: GND -> /GND
- Q1 pad 3: NET_Q1_DRAIN -> /LED_K
Routing:
- net /GND: track 0.00 -> 413.2 mm, vias 0 -> 11
- net GND: track 336.6 -> 0.00 mm, vias 4 -> 0
- net /3V3: track 0.00 -> 241.2 mm, vias 0 -> 8
- net VREF: track 226.6 -> 0.00 mm, vias 6 -> 0
- net 3V3_ANALOG: track 217.4 -> 0.00 mm, vias 9 -> 0
- net 3V3: track 182.2 -> 0.00 mm, vias 4 -> 0
- net /VREF: track 0.00 -> 171.4 mm, vias 0 -> 13
- net /3V3_ANALOG: track 0.00 -> 159.9 mm, vias 0 -> 8
- net /VTH_ON: track 0.00 -> 118.6 mm, vias 0 -> 7
- net /RAW_OFF_TL: track 0.00 -> 107.5 mm, vias 0 -> 4
- net /VTH_OFF: track 0.00 -> 106.1 mm, vias 0 -> 6
- net VPHOTO_TR: track 94.2 -> 0.00 mm, vias 3 -> 0
- net VPHOTO_TL: track 88.9 -> 0.00 mm, vias 1 -> 0
- net VTH_ON: track 86.8 -> 0.00 mm, vias 4 -> 0
- net /RAW_ON_TR: track 0.00 -> 86.0 mm, vias 0 -> 5
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- added copper zone on B.Cu, net /GND
- added copper zone on F.Cu, net /GND
- removed copper zone on B.Cu, net GND
- removed copper zone on F.Cu, net GND
Other:
- rule pad_to_mask_clearance: 0.05 -> 0
- board text removed: "BL"
- board text removed: "BR"
- board text removed: "OPTICAL BARRIER KEEP-OUT"
- board text removed: "REV A - NEUROMORPHIC IR SENSOR"
- board text removed: "TL"
- board text removed: "TR"
