File: neuromorphic-ir-event-sensor.kicad_sch (KiCad schematic)
At the start: 116 parts, among them Q1 AO3400A

Commit message: fix(pcb): correct LED1 pinout, complete routing, and regenerate manufacturing package
- Correct TSAL6200 IR LED pinout (Pad 1 Cathode -> LED_K, Pad 2 Anode -> 3V3) in schematic and PCB layout
- Complete copper routing with 0 DRC violations and 0 unconnected nets
- Re-export all production Gerbers, Excellon drill files, and revA ZIP archive
- Regenerate 3D CAD STEP model and documentation vector SVGs (PCB 2D & schematic)
Connections:
- net 3V3: now also LED1.2 (A)
- net LED_K: now also LED1.1 (K); no longer LED1.2 (A)
