File: neuromorphic-ir-event-sensor.kicad_sch (KiCad schematic)
At the start: 116 parts, among them Q1 AO3400A

Commit message: Promote verified Rev A candidate to main KiCad project
Parts:
- removed CA1, CA2, CA3, CA4, CREF2, C_DEC_CMP1, C_DEC_CMP2, C_DEC_CMP3, C_DEC_CMP4, C_DEC_TIA1, C_DEC_TIA2, C_DEC_TIA3, C_DEC_TIA4: 100nF, Capacitor_SMD:C_0603_1608Metric, symbol Device:C
- removed CF1, CF2, CF3, CF4: 47pF C0G, Capacitor_SMD:C_0603_1608Metric, symbol Device:C
- removed COS_OFF_BL, COS_OFF_BR, COS_OFF_TL, COS_OFF_TR, COS_ON_BL, COS_ON_BR, COS_ON_TL, COS_ON_TR: 12nF, Capacitor_SMD:C_0603_1608Metric, symbol Device:C
- removed CREF1: 1uF, Capacitor_SMD:C_0603_1608Metric, symbol Device:C
- removed C_BULK_A, C_BULK_D, C_LED: 10uF, Capacitor_SMD:C_0805_2012Metric, symbol Device:C
- removed DPD1, DPD2, DPD3, DPD4: VBPW34FASR, OptoDevice:Osram_BPW34S-SMD, symbol Sensor_Optical:BPW34-SMD
- removed J_DEBUG: Analog_Debug, Connector_PinHeader_2.54mm:PinHeader_1x06_P2.54mm_Vertical, symbol Connector_Generic:Conn_01x06
- removed J_FPGA: Tang_Nano_Event_Out, Connector_PinHeader_2.54mm:PinHeader_2x05_P2.54mm_Vertical, symbol Connector_Generic:Conn_02x05_Odd_Even
- removed LED1: TSAL6200, LED_THT:LED_D5.0mm, symbol Device:LED
- removed Q1: AO3400A, Package_TO_SOT_SMD:SOT-23, symbol Device:Q_NMOS
- removed RA1, RA2, RA3, RA4: 22k, Resistor_SMD:R_0603_1608Metric, symbol Device:R
- removed RF1, RF2, RF3, RF4: 18.0k 0.1%, Resistor_SMD:R_0603_1608Metric, symbol Device:R
- removed RG: 100R, Resistor_SMD:R_0603_1608Metric, symbol Device:R
- removed RLED: 82R 1206, Resistor_SMD:R_1206_3216Metric, symbol Device:R
- removed ROS_OFF_BL, ROS_OFF_BR, ROS_OFF_TL, ROS_OFF_TR, ROS_ON_BL, ROS_ON_BR, ROS_ON_TL, ROS_ON_TR: 8.2k, Resistor_SMD:R_0603_1608Metric, symbol Device:R
- removed ROUT_OFF_BL, ROUT_OFF_BR, ROUT_OFF_TL, ROUT_OFF_TR, ROUT_ON_BL, ROUT_ON_BR, ROUT_ON_TL, ROUT_ON_TR: 150R, Resistor_SMD:R_0603_1608Metric, symbol Device:R
- removed RPD: 100k, Resistor_SMD:R_0603_1608Metric, symbol Device:R
- removed RTHN_A: 301k 0.1%, Resistor_SMD:R_0603_1608Metric, symbol Device:R
- removed RTHN_B, RTHP_B: 10.0k 0.1%, Resistor_SMD:R_0603_1608Metric, symbol Device:R
- removed RTHP_A: 499k 0.1%, Resistor_SMD:R_0603_1608Metric, symbol Device:R
- removed TP_3V3: 3V3, TestPoint:TestPoint_Pad_D1.0mm, symbol Connector:TestPoint
- removed TP_3V3_ANALOG: 3V3_ANALOG, TestPoint:TestPoint_Pad_D1.0mm, symbol Connector:TestPoint
- removed TP_GND: GND, TestPoint:TestPoint_Pad_D1.0mm, symbol Connector:TestPoint
- removed TP_RAW_OFF_BL: RAW_OFF_BL, TestPoint:TestPoint_Pad_D1.0mm, symbol Connector:TestPoint
- removed TP_RAW_OFF_BR: RAW_OFF_BR, TestPoint:TestPoint_Pad_D1.0mm, symbol Connector:TestPoint
- removed TP_RAW_OFF_TL: RAW_OFF_TL, TestPoint:TestPoint_Pad_D1.0mm, symbol Connector:TestPoint
- removed TP_RAW_OFF_TR: RAW_OFF_TR, TestPoint:TestPoint_Pad_D1.0mm, symbol Connector:TestPoint
- removed TP_RAW_ON_BL: RAW_ON_BL, TestPoint:TestPoint_Pad_D1.0mm, symbol Connector:TestPoint
- removed TP_RAW_ON_BR: RAW_ON_BR, TestPoint:TestPoint_Pad_D1.0mm, symbol Connector:TestPoint
- removed TP_RAW_ON_TL: RAW_ON_TL, TestPoint:TestPoint_Pad_D1.0mm, symbol Connector:TestPoint
- removed TP_RAW_ON_TR: RAW_ON_TR, TestPoint:TestPoint_Pad_D1.0mm, symbol Connector:TestPoint
- removed TP_SPIKE_OFF_BL: SPIKE_OFF_BL, TestPoint:TestPoint_Pad_D1.0mm, symbol Connector:TestPoint
- removed TP_SPIKE_OFF_BR: SPIKE_OFF_BR, TestPoint:TestPoint_Pad_D1.0mm, symbol Connector:TestPoint
- removed TP_SPIKE_OFF_TL: SPIKE_OFF_TL, TestPoint:TestPoint_Pad_D1.0mm, symbol Connector:TestPoint
- removed TP_SPIKE_OFF_TR: SPIKE_OFF_TR, TestPoint:TestPoint_Pad_D1.0mm, symbol Connector:TestPoint
- removed TP_SPIKE_ON_BL: SPIKE_ON_BL, TestPoint:TestPoint_Pad_D1.0mm, symbol Connector:TestPoint
- removed TP_SPIKE_ON_BR: SPIKE_ON_BR, TestPoint:TestPoint_Pad_D1.0mm, symbol Connector:TestPoint
- removed TP_SPIKE_ON_TL: SPIKE_ON_TL, TestPoint:TestPoint_Pad_D1.0mm, symbol Connector:TestPoint
- removed TP_SPIKE_ON_TR: SPIKE_ON_TR, TestPoint:TestPoint_Pad_D1.0mm, symbol Connector:TestPoint
- removed TP_VEVENT_BL: VEVENT_BL, TestPoint:TestPoint_Pad_D1.0mm, symbol Connector:TestPoint
- removed TP_VEVENT_BR: VEVENT_BR, TestPoint:TestPoint_Pad_D1.0mm, symbol Connector:TestPoint
- removed TP_VEVENT_TL: VEVENT_TL, TestPoint:TestPoint_Pad_D1.0mm, symbol Connector:TestPoint
- removed TP_VEVENT_TR: VEVENT_TR, TestPoint:TestPoint_Pad_D1.0mm, symbol Connector:TestPoint
- removed TP_VPHOTO_BL: VPHOTO_BL, TestPoint:TestPoint_Pad_D1.0mm, symbol Connector:TestPoint
- removed TP_VPHOTO_BR: VPHOTO_BR, TestPoint:TestPoint_Pad_D1.0mm, symbol Connector:TestPoint
- removed TP_VPHOTO_TL: VPHOTO_TL, TestPoint:TestPoint_Pad_D1.0mm, symbol Connector:TestPoint
- removed TP_VPHOTO_TR: VPHOTO_TR, TestPoint:TestPoint_Pad_D1.0mm, symbol Connector:TestPoint
- removed TP_VREF: VREF, TestPoint:TestPoint_Pad_D1.0mm, symbol Connector:TestPoint
- removed TP_VTH_OFF: VTH_OFF, TestPoint:TestPoint_Pad_D1.0mm, symbol Connector:TestPoint
- removed TP_VTH_ON: VTH_ON, TestPoint:TestPoint_Pad_D1.0mm, symbol Connector:TestPoint
- removed U_CMP1, U_CMP2, U_CMP3, U_CMP4: TLV3202AIDR, Package_SO:SOIC-8_3.9x4.9mm_P1.27mm, symbol Comparator:LM393
- removed U_OS_OFF_BL, U_OS_OFF_BR, U_OS_OFF_TL, U_OS_OFF_TR, U_OS_ON_BL, U_OS_ON_BR, U_OS_ON_TL, U_OS_ON_TR: 74LVC1G123, Package_SO:VSSOP-8_2.3x2mm_P0.5mm, symbol 74xGxx:74LVC1G123
- removed U_REF: REF3312AIDBZR, Package_TO_SOT_SMD:SOT-23-3, symbol Reference_Voltage:REF3012
- removed U_TIA1, U_TIA2, U_TIA3, U_TIA4: OPA381AIDGKR, Package_SO:MSOP-8_3x3mm_P0.65mm, symbol Amplifier_Operational:OPA197xDGK
- added C1, C2, C3, C4: 47pF, Capacitor_SMD:C_0603_1608Metric, symbol Device:C
- added C10, C11, C12, C13, C14, C15, C16, C26, C30, C31, C32, C33, C34, C35, C36, C37, C5, C6, C7, C8, C9: 100nF, Capacitor_SMD:C_0603_1608Metric, symbol Device:C
- added C17, C18, C19, C20, C21, C22, C23, C24: 12nF, Capacitor_SMD:C_0603_1608Metric, symbol Device:C
- added C25: 1uF, Capacitor_SMD:C_0603_1608Metric, symbol Device:C
- added C27, C28, C29: 10uF, Capacitor_SMD:C_0805_2012Metric, symbol Device:C
- added D1, D2, D3, D4: VBPW34S, VBPW34S:XDCR_VBPW34S, symbol VBPW34S:VBPW34S
- added D5: TSAL6200, LED_THT:LED_D5.0mm, symbol Device:LED
- added H1, H2, H3, H4: MountingHole, MountingHole:MountingHole_3.2mm_M3, symbol Mechanical:MountingHole
- added H5, H6: MountingHole, MountingHole:MountingHole_2.2mm_M2, symbol Mechanical:MountingHole
- added J1: FPGA_Events_2x5, Connector_PinHeader_2.54mm:PinHeader_2x05_P2.54mm_Vertical, symbol Connector_Generic:Conn_02x05_Odd_Even
- added J2: Analog_Debug, Connector_PinHeader_2.54mm:PinHeader_1x06_P2.54mm_Vertical, symbol Connector_Generic:Conn_01x06
- added J3: LED_Enable_Input, Connector_PinHeader_2.54mm:PinHeader_1x02_P2.54mm_Vertical, symbol Connector_Generic:Conn_01x02
- added Q1: AO3400A, Package_TO_SOT_SMD:SOT-23, symbol Transistor_FET:AO3400A
- added R1, R2, R3, R4: 18.0k, Resistor_SMD:R_0603_1608Metric, symbol Device:R
- added R10, R11, R12, R13, R14, R15, R16, R9: 8.2k, Resistor_SMD:R_0603_1608Metric, symbol Device:R
- added R17, R18, R19, R20, R21, R22, R23, R24: 150R, Resistor_SMD:R_0603_1608Metric, symbol Device:R
- added R25: 82R, Resistor_SMD:R_1206_3216Metric, symbol Device:R
- added R26: 100R, Resistor_SMD:R_0603_1608Metric, symbol Device:R
- added R27: 100k, Resistor_SMD:R_0603_1608Metric, symbol Device:R
- added R28: 499k, Resistor_SMD:R_0603_1608Metric, symbol Device:R
- added R29, R30, R40, R41, R42, R43: 10.0k, Resistor_SMD:R_0603_1608Metric, symbol Device:R
- added R31: 301k, Resistor_SMD:R_0603_1608Metric, symbol Device:R
- added R32, R33, R34, R35, R36, R37, R38, R39: 2.0M, Resistor_SMD:R_0603_1608Metric, symbol Device:R
- added R5, R6, R7, R8: 22k, Resistor_SMD:R_0603_1608Metric, symbol Device:R
- added TP1: VTH_ON, TestPoint:TestPoint_Pad_D1.0mm, symbol Connector:TestPoint
- added TP10: RAW_OFF_BR, TestPoint:TestPoint_Pad_D1.0mm, symbol Connector:TestPoint
- added TP2: VTH_OFF, TestPoint:TestPoint_Pad_D1.0mm, symbol Connector:TestPoint
- added TP3: RAW_ON_TL, TestPoint:TestPoint_Pad_D1.0mm, symbol Connector:TestPoint
- added TP4: RAW_OFF_TL, TestPoint:TestPoint_Pad_D1.0mm, symbol Connector:TestPoint
- added TP5: RAW_ON_TR, TestPoint:TestPoint_Pad_D1.0mm, symbol Connector:TestPoint
- added TP6: RAW_OFF_TR, TestPoint:TestPoint_Pad_D1.0mm, symbol Connector:TestPoint
- added TP7: RAW_ON_BL, TestPoint:TestPoint_Pad_D1.0mm, symbol Connector:TestPoint
- added TP8: RAW_OFF_BL, TestPoint:TestPoint_Pad_D1.0mm, symbol Connector:TestPoint
- added TP9: RAW_ON_BR, TestPoint:TestPoint_Pad_D1.0mm, symbol Connector:TestPoint
- added U1, U2, U3, U4: OPA381AIDGKR, Package_SO:MSOP-8_3x3mm_P0.65mm, symbol Amplifier_Operational:OPA197xDGK
- added U10, U11, U12, U13, U14, U15, U16, U9: SN74LVC1G123DCU, Package_SO:VSSOP-8_2.3x2mm_P0.5mm, symbol 74xGxx:74LVC1G123
- added U17: REF3312AIDBZR, Package_TO_SOT_SMD:SOT-23-3, symbol Reference_Voltage:REF3012
- added U5, U6, U7, U8: TLV3202AIDR, Package_SO:SOIC-8_3.9x4.9mm_P1.27mm, symbol Comparator:MCP6562
- FB1: Function (none) -> Analog supply filter; MPN (none) -> BLM18AG601SN1D
Connections:
- net 3V3: now also C28.1, C29.1, C30.1, C31.1, C32.1, C33.1, C34.1, C35.1, C36.1, C37.1, J1.2 (Pin_2), R10.1, R11.1, R12.1, R13.1, R14.1, R15.1, R16.1, R25.1, R9.1, U10.3 (~{CLR}), U10.8 (VCC), U11.3 (~{CLR}), U11.8 (VCC), U12.3 (~{CLR}), U12.8 (VCC), U13.3 (~{CLR}), U13.8 (VCC), U14.3 (~{CLR}), U14.8 (VCC), U15.3 (~{CLR}), U15.8 (VCC), U16.3 (~{CLR}), U16.8 (VCC), U9.3 (~{CLR}), U9.8 (VCC)
- net 3V3_ANALOG: now also C10.1, C11.1, C12.1, C13.1, C14.1, C15.1, C16.1, C27.1, C9.1, R28.1, U1.7 (V+), U17.1 (IN), U2.7 (V+), U3.7 (V+), U4.7 (V+), U5.8 (V+), U6.8 (V+), U7.8 (V+), U8.8 (V+)
- net GND: now also C10.2, C11.2, C12.2, C13.2, C14.2, C15.2, C16.2, C25.2, C26.2, C27.2, C28.2, C29.2, C30.2, C31.2, C32.2, C33.2, C34.2, C35.2, C36.2, C37.2, C9.2, D1.A, D2.A, D3.A, D4.A, J1.1 (Pin_1), J2.1 (Pin_1), J3.2 (Pin_2), Q1.2 (S), R27.2, R31.2, U1.4 (V-), U10.1 (~{A}), U10.4 (GND), U11.1 (~{A}), U11.4 (GND), U12.1 (~{A}), U12.4 (GND), U13.1 (~{A}), U13.4 (GND), U14.1 (~{A}), U14.4 (GND), U15.1 (~{A}), U15.4 (GND), U16.1 (~{A}), U16.4 (GND), U17.3 (GND), U2.4 (V-), U3.4 (V-), U4.4 (V-), U5.4 (V-), U6.4 (V-), U7.4 (V-), U8.4 (V-), U9.1 (~{A}), U9.4 (GND)
- net LED_EN: now also J3.1 (Pin_1), R26.1
- net LED_GATE: now also Q1.1 (G), R26.2, R27.1
- net LED_K: now also D5.1 (K), Q1.3 (D)
- net RAW_OFF_BL: now also R37.1, TP8.1, U14.2 (B), U7.7
- net RAW_OFF_BR: now also R39.1, TP10.1, U16.2 (B), U8.7
- net RAW_OFF_TL: now also R33.1, TP4.1, U10.2 (B), U5.7
- net RAW_OFF_TR: now also R35.1, TP6.1, U12.2 (B), U6.7
- net RAW_ON_BL: now also R36.1, TP7.1, U13.2 (B), U7.1
- net RAW_ON_BR: now also R38.1, TP9.1, U15.2 (B), U8.1
- net RAW_ON_TL: now also R32.1, TP3.1, U5.1, U9.2 (B)
- net RAW_ON_TR: now also R34.1, TP5.1, U11.2 (B), U6.1
- net SPIKE_OFF_BL: now also J1.8 (Pin_8), R22.2
- net SPIKE_OFF_BR: now also J1.10 (Pin_10), R24.2
- net SPIKE_OFF_TL: now also J1.4 (Pin_4), R18.2
- net SPIKE_OFF_TR: now also J1.6 (Pin_6), R20.2
- net SPIKE_ON_BL: now also J1.7 (Pin_7), R21.2
- net SPIKE_ON_BR: now also J1.9 (Pin_9), R23.2
- net SPIKE_ON_TL: now also J1.3 (Pin_3), R17.2
- net SPIKE_ON_TR: now also J1.5 (Pin_5), R19.2
- net VEVENT_BL: now also C7.2, R36.2, R7.1, U7.3 (+), U7.6 (-)
- net VEVENT_BR: now also C8.2, R38.2, R8.1, U8.3 (+), U8.6 (-)
- net VEVENT_TL: now also C5.2, R32.2, R5.1, U5.3 (+), U5.6 (-)
- net VEVENT_TR: now also C6.2, R34.2, R6.1, U6.3 (+), U6.6 (-)
- net VPHOTO_BL: now also C3.2, C7.1, J2.5 (Pin_5), R3.2, U3.6
- net VPHOTO_BR: now also C4.2, C8.1, J2.6 (Pin_6), R4.2, U4.6
- net VPHOTO_TL: now also C1.2, C5.1, J2.3 (Pin_3), R1.2, U1.6
- net VPHOTO_TR: now also C2.2, C6.1, J2.4 (Pin_4), R2.2, U2.6
- net VREF: now also C25.1, C26.1, J2.2 (Pin_2), R29.2, R30.1, R5.2, R6.2, R7.2, R8.2, U1.3 (+), U17.2 (OUT), U2.3 (+), U3.3 (+), U4.3 (+)
- net VTH_OFF: now also R30.2, R31.1, R40.1, R41.1, R42.1, R43.1, TP2.1
- net VTH_ON: now also R28.2, R29.1, TP1.1, U5.2 (-), U6.2 (-), U7.2 (-), U8.2 (-)
- new net CEXT_OFF_BL: C22.1, U14.6 (Cext)
- new net CEXT_OFF_BR: C24.1, U16.6 (Cext)
- new net CEXT_OFF_TL: C18.1, U10.6 (Cext)
- new net CEXT_OFF_TR: C20.1, U12.6 (Cext)
- new net CEXT_ON_BL: C21.1, U13.6 (Cext)
- new net CEXT_ON_BR: C23.1, U15.6 (Cext)
- new net CEXT_ON_TL: C17.1, U9.6 (Cext)
- new net CEXT_ON_TR: C19.1, U11.6 (Cext)
- new net LED_A: D5.2 (A), R25.2
- new net OS_OUT_OFF_BL: R22.1, U14.5 (Q)
- new net OS_OUT_OFF_BR: R24.1, U16.5 (Q)
- new net OS_OUT_OFF_TL: R18.1, U10.5 (Q)
- new net OS_OUT_OFF_TR: R20.1, U12.5 (Q)
- new net OS_OUT_ON_BL: R21.1, U13.5 (Q)
- new net OS_OUT_ON_BR: R23.1, U15.5 (Q)
- new net OS_OUT_ON_TL: R17.1, U9.5 (Q)
- new net OS_OUT_ON_TR: R19.1, U11.5 (Q)
- new net REXT_OFF_BL: C22.2, R14.2, U14.7 (RCext)
- new net REXT_OFF_BR: C24.2, R16.2, U16.7 (RCext)
- new net REXT_OFF_TL: C18.2, R10.2, U10.7 (RCext)
- new net REXT_OFF_TR: C20.2, R12.2, U12.7 (RCext)
- new net REXT_ON_BL: C21.2, R13.2, U13.7 (RCext)
- new net REXT_ON_BR: C23.2, R15.2, U15.7 (RCext)
- new net REXT_ON_TL: C17.2, R9.2, U9.7 (RCext)
- new net REXT_ON_TR: C19.2, R11.2, U11.7 (RCext)
- new net TIA_IN_BL: C3.1, D3.K, R3.1, U3.2 (-)
- new net TIA_IN_BR: C4.1, D4.K, R4.1, U4.2 (-)
- new net TIA_IN_TL: C1.1, D1.K, R1.1, U1.2 (-)
- new net TIA_IN_TR: C2.1, D2.K, R2.1, U2.2 (-)
- new net VTH_OFF_BL: R37.2, R42.2, U7.5 (+)
- new net VTH_OFF_BR: R39.2, R43.2, U8.5 (+)
- new net VTH_OFF_TL: R33.2, R40.2, U5.5 (+)
- new net VTH_OFF_TR: R35.2, R41.2, U6.5 (+)
- no-connect marks 0 -> 12
Other:
- note added: "Circuit"
- note added: "Design specification plus user decisions: 10-pin event header, VBPW34S, FPGA-controlled LED_EN. Nominal VTH_ON 1.2903 V and VTH_OFF 1.2098 V at 3.300/1.250 V; R28-R31 0.1%. This candidate is not yet fabrication approved."
- note added: "Power flags"
- company: Open SNN Robot Project -> (none)
- title: Rev A Neuromorphic IR Event Sensor -> Neuromorphic IR Event Sensor
